File: pcb/manjaro_mx.kicad_pcb (KiCad board)
At the start: 2 copper layers, 286.5 x 118.5 mm, 111 parts, among them J2 MJ-4PP-9, SW1 SW_Push, SW10 SW_Push, SW11 SW_Push, SW12 SW_Push, SW13 SW_Push, SW14 SW_Push, SW15 SW_Push, SW16 SW_Push, SW17 SW_Push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

Commit message: [base] layout 7x4 with RP2040 MCU
Parts:
- removed ? (x10): , 
- removed BT1, rBT1: Battery_Cell, Connector_JST:JST_PH_S2B-PH-K_1x02_P2.00mm_Horizontal
- removed EXSW1, rEXSW1: RotaryEncoder_Switch, Keebio-Parts:RotaryEncoder_EC11
- removed PowerSW1, rPowerSW1: SW_Wuerth_450301014042, Button_Switch_THT:SW_Slide-03_Wuerth-WS-SLTV_10x2.5x6.4_P2.54mm
- removed U1, rU1: nice_nano, nice-nano-kicad:nice_nano
- removed rJ3: Conn_01x06, Connector_PinHeader_2.54mm:PinHeader_1x06_P2.54mm_Vertical
- added D25: 1N4148WT, Keebio-Parts:D_SOD-323, B.Cu at (107.2, 112.2)
- added D26: 1N4148WT, Keebio-Parts:D_SOD-323, B.Cu at (88.1, 112.2)
- added D27: 1N4148WT, Keebio-Parts:D_SOD-323, B.Cu at (69.0, 112.2)
- added D28: 1N4148WT, Keebio-Parts:D_SOD-323, B.Cu at (50.0, 112.2)
- added RZ1: RP2040-Zero, rp2040-zero-kicad:RP2040-Zero, F.Cu at (155.7, 39.6)
- added SW25: SW_Push, kbd:keyswitch_cherrymx_hotswap_1u, B.Cu at (107.2, 107.2)
- added SW26: SW_Push, kbd:keyswitch_cherrymx_hotswap_1u, B.Cu at (88.1, 107.2)
- added SW27: SW_Push, kbd:keyswitch_cherrymx_hotswap_1u, B.Cu at (69.0, 107.2)
- added SW28: SW_Push, kbd:keyswitch_cherrymx_hotswap_1u, B.Cu at (50.0, 107.2)
- added rD22: 1N4148WT, Keebio-Parts:D_SOD-323, B.Cu at (210.9, 102.2)
- added rD23: 1N4148WT, Keebio-Parts:D_SOD-323, B.Cu at (230.0, 102.2)
- added rD24: 1N4148WT, Keebio-Parts:D_SOD-323, B.Cu at (249.1, 102.2)
- added rD25: 1N4148WT, Keebio-Parts:D_SOD-323, B.Cu at (268.1, 112.2)
- added rD26: 1N4148WT, Keebio-Parts:D_SOD-323, B.Cu at (287.1, 112.2)
- added rD27: 1N4148WT, Keebio-Parts:D_SOD-323, B.Cu at (306.2, 112.2)
- added rD28: 1N4148WT, Keebio-Parts:D_SOD-323, B.Cu at (325.2, 112.2)
- added rRZ1: RP2040-Zero, rp2040-zero-kicad:RP2040-Zero, F.Cu at (201.7, 39.5)
- added rSW22: SW_Push, kbd:keyswitch_choc12_hotswap_1u, B.Cu at (210.9, 107.2)
- added rSW23: SW_Push, kbd:keyswitch_choc12_hotswap_1u, B.Cu at (230.0, 107.2)
- added rSW24: SW_Push, kbd:keyswitch_choc12_hotswap_1u, B.Cu at (249.1, 107.2)
- added rSW25: SW_Push, kbd:keyswitch_cherrymx_hotswap_1u, B.Cu at (268.1, 107.2)
- added rSW26: SW_Push, kbd:keyswitch_cherrymx_hotswap_1u, B.Cu at (287.1, 107.2)
- added rSW27: SW_Push, kbd:keyswitch_cherrymx_hotswap_1u, B.Cu at (306.2, 107.2)
- added rSW28: SW_Push, kbd:keyswitch_cherrymx_hotswap_1u, B.Cu at (325.2, 107.2)
- SW22, SW23, SW24: footprint kbd:keyswitch_cherrymx_hotswap_1u -> kbd:keyswitch_choc12_hotswap_1u
- moved rD7 120.9 mm to (325.2, 55.0), turned to 0 degrees
- moved rSW7 115.7 mm to (325.2, 50.0)
- moved rD19 109.1 mm to (287.1, 93.1), turned to 0 degrees
- moved rD20 105.8 mm to (306.2, 93.1), turned to 0 degrees
- moved rSW19 105.7 mm to (287.1, 88.1), turned to 180 degrees
- moved rD13 103.0 mm to (306.2, 74.0), turned to 0 degrees
- moved rD14 102.3 mm to (325.2, 74.0), turned to 0 degrees
- moved D7 102.1 mm to (50.0, 55.0), turned to 0 degrees
- moved rSW20 101.7 mm to (306.2, 88.1), turned to 180 degrees
- moved rSW13 97.9 mm to (306.2, 69.0)
- moved rSW14 97.1 mm to (325.2, 69.0)
- moved SW7 97.0 mm to (50.0, 50.0)
- moved D19 92.1 mm to (88.1, 93.1), turned to 0 degrees
- moved SW19 88.6 mm to (88.1, 88.1), turned to 180 degrees
- moved D20 88.4 mm to (69.0, 93.1), turned to 0 degrees
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Connections:
- D13 pad 1: ROW2 -> ROW1
- D14 pad 1: ROW2 -> ROW1
- D19 pad 1: ROW3 -> ROW2
- D20 pad 1: ROW3 -> ROW2
- D21 pad 1: ROW3 -> ROW2
- D7 pad 1: ROW1 -> ROW0
- J2 pad 3: BAT- -> GND
- SW10 pad 1: COL3 -> COL2
- SW11 pad 1: COL4 -> COL3
- SW12 pad 1: COL5 -> COL4
- SW13 pad 1: COL0 -> COL5
- SW14 pad 1: COL1 -> COL6
- SW15 pad 1: COL2 -> COL0
- SW16 pad 1: COL3 -> COL1
- SW17 pad 1: COL4 -> COL2
- SW18 pad 1: COL5 -> COL3
- SW19 pad 1: COL0 -> COL4
- SW20 pad 1: COL1 -> COL5
- SW21 pad 1: COL2 -> COL6
- SW22 pad 1: COL3 -> COL0
- SW23 pad 1: COL4 -> COL1
- SW24 pad 1: COL5 -> COL2
- SW7 pad 1: COL0 -> COL6
- SW8 pad 1: COL1 -> COL0
- SW9 pad 1: COL2 -> COL1
- rD13 pad 1: rROW2 -> rROW1
- rD14 pad 1: rROW2 -> rROW1
- rD19 pad 1: rROW3 -> rROW2
- rD20 pad 1: rROW3 -> rROW2
- rD21 pad 1: rROW3 -> rROW2
- rD7 pad 1: rROW1 -> rROW0
- rJ2 pad 3: rBAT- -> rGND
- rSW10 pad 2: rCOL3 -> rCOL2
- rSW11 pad 2: rCOL4 -> rCOL3
- rSW12 pad 2: rCOL5 -> rCOL4
- rSW13 pad 2: rCOL0 -> rCOL5
- rSW14 pad 2: rCOL1 -> rCOL6
- rSW15 pad 2: rCOL2 -> rCOL0
- rSW16 pad 2: rCOL3 -> rCOL1
- rSW17 pad 2: rCOL4 -> rCOL2
- rSW18 pad 2: rCOL5 -> rCOL3
- rSW19 pad 2: rCOL0 -> rCOL4
- rSW20 pad 2: rCOL1 -> rCOL5
- rSW21 pad 2: rCOL2 -> rCOL6
- rSW7 pad 2: rCOL0 -> rCOL6
- rSW8 pad 2: rCOL1 -> rCOL0
- rSW9 pad 2: rCOL2 -> rCOL1
Routing:
- net rBAT-: track 311.2 -> 0.00 mm, vias 1 -> 0
- net rROW3: track 229.2 -> 0.00 mm, vias 1 -> 0
- net ROW3: track 218.9 -> 0.00 mm, vias 1 -> 0
- net BAT-: track 212.9 -> 0.00 mm, vias 3 -> 0
- net ROW2: track 199.5 -> 0.00 mm, vias 1 -> 0
- net DATA: track 192.5 -> 0.00 mm
- net rROW2: track 184.7 -> 0.00 mm, vias 1 -> 0
- net ROW1: track 180.6 -> 0.00 mm, vias 1 -> 0
- net rDATA: track 178.1 -> 0.00 mm, vias 2 -> 0
- net rVCC: track 175.2 -> 0.00 mm, vias 3 -> 0
- net VCC: track 174.7 -> 0.00 mm
- net COL0: track 173.9 -> 0.00 mm, vias 8 -> 0
- net REB: track 168.0 -> 0.00 mm, vias 2 -> 0
- net rKEYEX1: track 167.3 -> 0.00 mm
- net rCOL0: track 166.0 -> 0.00 mm, vias 6 -> 0
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Other:
- board outline removed
- board text removed: "+"
- board text removed: "-"
- board text removed: "Manjaro v1"
- board text removed: "On"
